Commit message: upgrade urdf model

File: src/URDF_Gyrosse_description/urdf/URDF_Gyrosse.xacro (robot description, xacro)
@@ -2,11 +2,13 @@
 <robot name="URDF_Gyrosse" xmlns:xacro="http://www.ros.org/wiki/xacro">
 <xacro:include filename="$(find URDF_Gyrosse_description)/urdf/materials.xacro" />
-<xacro:include filename="$(find URDF_Gyrosse_description)/urdf/URDF_Gyrosse.trans" />
+<xacro:include filename="$(find URDF_Gyrosse_description)/urdf/URDF_Gyrosse.control" />
 <xacro:include filename="$(find URDF_Gyrosse_description)/urdf/URDF_Gyrosse.gazebo" />
-<link name="base_link">
+ <link name="base_link" />
+<!-- Chassis -->
+<link name="chassis">
   <inertial>
     <origin xyz="0.19050000000000009 -0.007676917492127958 -0.0014829191458506099" rpy="0 0 0"/>
     <mass value="13.254937098226266"/>
-    <inertia ixx="0.132414" iyy="0.271154" izz="0.221585" ixy="-0.0" iyz="0.000151" ixz="-0.0"/>
+    <inertia ixx="0.132414" iyy="0.271154" izz="0.221585" ixy="0" iyz="0.000151" ixz="0"/>
   </inertial>
   <visual>
@@ -24,107 +26,116 @@
   </collision>
 </link>
-<link name="wheel_right_1">
+<joint name="chassis_joint" type="fixed">
+  <origin xyz="0 0 0" rpy="0 0 0" />
+  <parent link="base_link" />
+  <child link="chassis" />
+</joint>
+<!-- right wheel Link -->
+<link name="right_wheel">
   <inertial>
     <origin xyz="-0.049489111284257994 -1.3199520432358287e-15 2.061614684425312e-16" rpy="0 0 0"/>
     <mass value="1.2625898797377435"/>
-    <inertia ixx="0.041938" iyy="0.021235" izz="0.021235" ixy="-0.0" iyz="-0.0" ixz="-0.0"/>
+    <inertia ixx="0.041938" iyy="0.021235" izz="0.021235" ixy="0" iyz="0" ixz="0"/>
   </inertial>
   <visual>
-    <origin xyz="-0.0 -0.0 -0.0" rpy="0 0 0"/>
+    <origin xyz="0 0 0" rpy="0 0 0"/>
     <geometry>
-      <mesh filename="file://$(find URDF_Gyrosse_description)/meshes/wheel_right_1.stl" scale="0.001 0.001 0.001"/>
+      <mesh filename="file://$(find URDF_Gyrosse_description)/meshes/right_wheel.stl" scale="0.001 0.001 0.001"/>
     </geometry>
-    <material name="silver"/>
+    <material name="Black"/>
   </visual>
   <collision>
-    <origin xyz="-0.0 -0.0 -0.0" rpy="0 0 0"/>
+    <origin xyz="0 0 0" rpy="0 0 0"/>
     <geometry>
-      <mesh filename="file://$(find URDF_Gyrosse_description)/meshes/wheel_right_1.stl" scale="0.001 0.001 0.001"/>
+      <mesh filename="file://$(find URDF_Gyrosse_description)/meshes/right_wheel.stl" scale="0.001 0.001 0.001"/>
     </geometry>
   </collision>
 </link>
-<link name="flywheel_right_1">
+<joint name="right_wheel_joint" type="continuous">
+  <origin xyz="0 0 0" rpy="0 0 0"/>
+  <parent link="chassis"/>
+  <child link="right_wheel"/>
+  <axis xyz="0 0 0"/>
+</joint>
+<!-- right flywheel Link -->
+<link name="right_flywheel">
   <inertial>
     <origin xyz="-0.008066340570656319 1.271316816228521e-16 1.7394980092897013e-16" rpy="0 0 0"/>
     <mass value="1.7384117767470415"/>
-    <inertia ixx="0.018431" iyy="0.009354" izz="0.009354" ixy="0.0" iyz="0.0" ixz="0.0"/>
+    <inertia ixx="0.018431" iyy="0.009354" izz="0.009354" ixy="0" iyz="0" ixz="0"/>
   </inertial>
   <visual>
-    <origin xyz="-0.108 -0.0 -0.0" rpy="0 0 0"/>
+    <origin xyz="-0.108 0 0" rpy="0 0 0"/>
     <geometry>
-      <mesh filename="file://$(find URDF_Gyrosse_description)/meshes/flywheel_right_1.stl" scale="0.001 0.001 0.001"/>
+      <mesh filename="file://$(find URDF_Gyrosse_description)/meshes/right_flywheel.stl" scale="0.001 0.001 0.001"/>
     </geometry>
-    <material name="silver"/>
+    <material name="Grey"/>
   </visual>
   <collision>
-    <origin xyz="-0.108 -0.0 -0.0" rpy="0 0 0"/>
+    <origin xyz="-0.108 0 0" rpy="0 0 0"/>
     <geometry>
-      <mesh filename="file://$(find URDF_Gyrosse_description)/meshes/flywheel_right_1.stl" scale="0.001 0.001 0.001"/>
+      <mesh filename="file://$(find URDF_Gyrosse_description)/meshes/right_flywheel.stl" scale="0.001 0.001 0.001"/>
     </geometry>
   </collision>
 </link>
-<link name="wheel_left_1">
+<joint name="right_flywheel_joint" type="continuous">
+  <origin xyz="0.108 0 0" rpy="0 0 0"/>
+  <parent link="chassis"/>
+  <child link="right_flywheel"/>
+  <axis xyz="1 0 0"/>
+</joint>
+  <!-- left wheel Link -->
+<link name="left_wheel">
   <inertial>
     <origin xyz="0.04948911128425798 -8.531713599697203e-16 -2.7715603505479613e-16" rpy="0 0 0"/>
     <mass value="1.2625898797377435"/>
-    <inertia ixx="0.041938" iyy="0.021235" izz="0.021235" ixy="0.0" iyz="-0.0" ixz="-0.0"/>
+    <inertia ixx="0.041938" iyy="0.021235" izz="0.021235" ixy="0" iyz="0" ixz="0"/>
   </inertial>
   <visual>
-    <origin xyz="-0.381 -0.0 -0.0" rpy="0 0 0"/>
+    <origin xyz="-0.381 0 0" rpy="0 0 0"/>
     <geometry>
-      <mesh filename="file://$(find URDF_Gyrosse_description)/meshes/wheel_left_1.stl" scale="0.001 0.001 0.001"/>
+      <mesh filename="file://$(find URDF_Gyrosse_description)/meshes/left_wheel.stl" scale="0.001 0.001 0.001"/>
     </geometry>
-    <material name="silver"/>
+    <material name="Black"/>
   </visual>
   <collision>
-    <origin xyz="-0.381 -0.0 -0.0" rpy="0 0 0"/>
+    <origin xyz="-0.381 0 0" rpy="0 0 0"/>
     <geometry>
-      <mesh filename="file://$(find URDF_Gyrosse_description)/meshes/wheel_left_1.stl" scale="0.001 0.001 0.001"/>
+      <mesh filename="file://$(find URDF_Gyrosse_description)/meshes/left_wheel.stl" scale="0.001 0.001 0.001"/>
     </geometry>
   </collision>
 </link>
-<link name="flywheel_left_1">
+<joint name="left_wheel_joint" type="continuous">
+  <origin xyz="0.381 0 0" rpy="0 0 0"/>
+  <parent link="base_link"/>
+  <child link="left_wheel"/>
+  <axis xyz="1 0 0"/>
+</joint>
+<!-- left flywheel Link -->
+<link name="left_flywheel">
   <inertial>
     <origin xyz="0.008066340570656305 1.553831664279304e-16 -1.0733641945145496e-16" rpy="0 0 0"/>
     <mass value="1.7384117767470415"/>
-    <inertia ixx="0.018431" iyy="0.009354" izz="0.009354" ixy="-0.0" iyz="-0.0" ixz="0.0"/>
+    <inertia ixx="0.018431" iyy="0.009354" izz="0.009354" ixy="0" iyz="0" ixz="0"/>
   </inertial>
   <visual>
-    <origin xyz="-0.273 -0.0 -0.0" rpy="0 0 0"/>
+    <origin xyz="-0.273 0 0" rpy="0 0 0"/>
     <geometry>
-      <mesh filename="file://$(find URDF_Gyrosse_description)/meshes/flywheel_left_1.stl" scale="0.001 0.001 0.001"/>
+      <mesh filename="file://$(find URDF_Gyrosse_description)/meshes/left_flywheel.stl" scale="0.001 0.001 0.001"/>
     </geometry>
-    <material name="silver"/>
+    <material name="Grey"/>
   </visual>
   <collision>
-    <origin xyz="-0.273 -0.0 -0.0" rpy="0 0 0"/>
+    <origin xyz="-0.273 0 0" rpy="0 0 0"/>
     <geometry>
-      <mesh filename="file://$(find URDF_Gyrosse_description)/meshes/flywheel_left_1.stl" scale="0.001 0.001 0.001"/>
+      <mesh filename="file://$(find URDF_Gyrosse_description)/meshes/left_flywheel.stl" scale="0.001 0.001 0.001"/>
     </geometry>
   </collision>
 </link>
-<joint name="wheel_right_to_base_link" type="continuous">
-  <origin xyz="0.0 0.0 0.0" rpy="0 0 0"/>
-  <parent link="base_link"/>
-  <child link="wheel_right_1"/>
-  <axis xyz="1.0 0.0 0.0"/>
-</joint>
-<joint name="flywheel_right_to_base_link" type="continuous">
-  <origin xyz="0.108 0.0 0.0" rpy="0 0 0"/>
-  <parent link="base_link"/>
-  <child link="flywheel_right_1"/>
-  <axis xyz="1.0 0.0 0.0"/>
-</joint>
-<joint name="wheel_left_to_base_link" type="continuous">
-  <origin xyz="0.381 0.0 0.0" rpy="0 0 0"/>
-  <parent link="base_link"/>
-  <child link="wheel_left_1"/>
-  <axis xyz="1.0 0.0 0.0"/>
-</joint>
-<joint name="flywheel_left_to_base_link" type="continuous">
-  <origin xyz="0.273 0.0 0.0" rpy="0 0 0"/>
-  <parent link="base_link"/>
-  <child link="flywheel_left_1"/>
-  <axis xyz="-1.0 0.0 0.0"/>
+<joint name="left_flywheel_joint" type="continuous">
+  <origin xyz="0.273 0 0" rpy="0 0 0"/>
+  <parent link="chassis"/>
+  <child link="left_flywheel"/>
+  <axis xyz="-1 0 0"/>
 </joint>
 </robot>

File: src/URDF_Gyrosse_description/urdf/materials.xacro (robot description, xacro)
@@ -4,3 +4,15 @@
   <color rgba="0.700 0.700 0.700 1.000"/>
 </material>
+ <material name="Black">
+    <color rgba="0 0 0 1" />
+  </material>
+  <material name="Grey">
+    <color rgba="0.8 0.8 0.8 1" />
+  </material>
+  <material name="Orange">
+    <color rgba="1 0.6 0 1" />
+  </material>
+  <material name="White">
+    <color rgba="1 1 1 1" />
+  </material>
 </robot>
